File: board/nano_mini_usb.sch (KiCad schematic (older format))
At the start: 22 parts, among them J1 Conn_01x04_Male, J2 Conn_01x04_Male, J3 Conn_01x02_Male, J4 Conn_01x02_Male, J5 Conn_01x02_Male, J6 Conn_01x04_Male, J7 Conn_01x03_Male, J8 Conn_01x02_Male, SW1 SW_DIP_x04

Commit message: Update PCB. Re-route switch power to Arduino +5V
Connections:
- net +5V: now also J8.1 (Pin_1); no longer J5.1 (Pin_1), J8.2 (Pin_2), SW1.1, SW1.2, SW1.3, SW1.4
- net arduino_pwr: now also SW1.1, SW1.2, SW1.3, SW1.4; no longer J8.1 (Pin_1)
- new net USB_pwr: J5.1 (Pin_1), J8.2 (Pin_2)
Changed lines of the file:
@@
 $EndComp
-Wire Wire Line
-	6400 2050 6400 2350
 Wire Wire Line
 	6200 4350 6200 4500
@@
 Wire Wire Line
 	3850 4900 4200 4900
-$Comp
-L power:+5V #PWR07
-U 1 1 61563939
-P 7650 3200
-F 0 "#PWR07" H 7650 3050 50  0001 C CNN
-F 1 "+5V" H 7665 3373 50  0000 C CNN
-F 2 "" H 7650 3200 50  0001 C CNN
-F 3 "" H 7650 3200 50  0001 C CNN
-	1    7650 3200
-	0    -1   -1   0
-$EndComp
 Wire Wire Line
 	7650 3200 7750 3200
@@
 Wire Wire Line
 	4100 5300 4200 5300
-Text GLabel 6400 2050 1    50   Input ~ 0
-arduino_pwr
-Text GLabel 4200 3800 2    50   Input ~ 0
-arduino_pwr
 $Comp
 L Connector:Conn_01x02_Male J8
@@
 $EndComp
 Wire Wire Line
-	3850 3800 4200 3800
-Wire Wire Line
 	3850 3900 4400 3900
-Wire Wire Line
-	4400 3900 4400 4000
 Wire Wire Line
 	4400 4150 3850 4150
@@
 Text GLabel 5600 3650 0    50   Input ~ 0
 LED2
+Text GLabel 7650 3200 0    50   Input ~ 0
+arduino_pwr
+Wire Wire Line
+	6400 2050 6400 2350
+Text GLabel 6400 2050 1    50   Input ~ 0
+arduino_pwr
 $Comp
 L power:+5V #PWR0101
 U 1 1 617ECCFA
-P 4500 4000
-F 0 "#PWR0101" H 4500 3850 50  0001 C CNN
-F 1 "+5V" V 4515 4128 50  0000 L CNN
-F 2 "" H 4500 4000 50  0001 C CNN
-F 3 "" H 4500 4000 50  0001 C CNN
-	1    4500 4000
-	0    1    1    0
-$EndComp
-Wire Wire Line
-	4400 4000 4500 4000
-Connection ~ 4400 4000
-Wire Wire Line
-	4400 4000 4400 4150
+P 4250 3700
+F 0 "#PWR0101" H 4250 3550 50  0001 C CNN
+F 1 "+5V" V 4265 3828 50  0000 L CNN
+F 2 "" H 4250 3700 50  0001 C CNN
+F 3 "" H 4250 3700 50  0001 C CNN
+	1    4250 3700
+	0    1    1    0
+$EndComp
+Wire Wire Line
+	4150 3700 4250 3700
+Wire Wire Line
+	4400 3900 4400 4150
+Wire Wire Line
+	4150 3700 4150 3800
+Wire Wire Line
+	3850 3800 4150 3800
+Wire Wire Line
+	4150 3800 4200 3800
+Connection ~ 4150 3800
 $EndSCHEMATC
